File: hardware/electronics/QMKMouse/Mechanical-SchDoc.kicad_sch (KiCad schematic)
At the start: 33 parts

Commit message: fix minor Schematic naming errors; improve BoM generation
Parts:
- HOLE.1, HOLE.2, MCH.FID.1, MCH.FID.2, MCH.LOGO.2, MCH.SP.1, MCH.SP.10, MCH.SP.11, MCH.SP.12, MCH.SP.13, MCH.SP.14, MCH.SP.15, MCH.SP.16, MCH.SP.17, MCH.SP.18, MCH.SP.19, MCH.SP.2, MCH.SP.20, MCH.SP.21, MCH.SP.22, MCH.SP.23, MCH.SP.24, MCH.SP.25, MCH.SP.26, MCH.SP.27, MCH.SP.28, MCH.SP.3, MCH.SP.4, MCH.SP.5, MCH.SP.6, MCH.SP.7, MCH.SP.8, MCH.SP.9: now left out of the parts list
Changed lines of the file:
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@@
   )
   (symbol (lib_name "Spark_gap_1") (lib_id "Mouse_Parts:Spark_gap") (at 180.34 109.22 0) (unit 1)
-    (in_bom yes) (on_board yes)
+    (in_bom no) (on_board yes)
     (property "Reference" "MCH.SP.18" (id 0) (at 175.26 102.87 0)
       (effects (font (size 1.27 1.27)) (justify left))
@@
   )
   (symbol (lib_name "Spark_gap_3") (lib_id "Mouse_Parts:Spark_gap") (at 187.96 109.22 0) (unit 1)
-    (in_bom yes) (on_board yes)
+    (in_bom no) (on_board yes)
     (property "Reference" "MCH.SP.19" (id 0) (at 182.88 105.41 0)
       (effects (font (size 1.27 1.27)) (justify left))
@@
   )
   (symbol (lib_name "Spark_gap_6") (lib_id "Mouse_Parts:Spark_gap") (at 170.18 83.82 0) (unit 1)
-    (in_bom yes) (on_board yes)
+    (in_bom no) (on_board yes)
     (property "Reference" "MCH.SP.7" (id 0) (at 165.1 80.01 0)
       (effects (font (size 1.27 1.27)) (justify left))
@@
   )
   (symbol (lib_name "Spark_gap_27") (lib_id "Mouse_Parts:Spark_gap") (at 187.96 134.62 0) (unit 1)
-    (in_bom yes) (on_board yes)
+    (in_bom no) (on_board yes)
     (property "Reference" "MCH.SP.28" (id 0) (at 182.88 130.81 0)
       (effects (font (size 1.27 1.27)) (justify left))
@@
   )
   (symbol (lib_id "Mouse_Parts:Fiducial") (at 73.66 53.34 0) (unit 1)
-    (in_bom yes) (on_board yes) (fields_autoplaced)
+    (in_bom no) (on_board yes) (fields_autoplaced)
     (property "Reference" "MCH.FID.2" (id 0) (at 76.2 52.0699 0)
       (effects (font (size 1.27 1.27)) (justify left))
@@
   )
   (symbol (lib_id "Mechanical:MountingHole") (at 74.93 69.85 0) (unit 1)
-    (in_bom yes) (on_board yes) (fields_autoplaced)
+    (in_bom no) (on_board yes) (fields_autoplaced)
     (property "Reference" "HOLE.2" (id 0) (at 77.47 68.5799 0)
       (effects (font (size 1.27 1.27)) (justify left))
@@
   )
   (symbol (lib_name "Spark_gap_13") (lib_id "Mouse_Parts:Spark_gap") (at 151.13 83.82 0) (unit 1)
-    (in_bom yes) (on_board yes)
+    (in_bom no) (on_board yes)
     (property "Reference" "MCH.SP.4" (id 0) (at 146.05 77.47 0)
       (effects (font (size 1.27 1.27)) (justify left))
@@
   )
   (symbol (lib_name "Spark_gap_5") (lib_id "Mouse_Parts:Spark_gap") (at 158.75 83.82 0) (unit 1)
-    (in_bom yes) (on_board yes)
+    (in_bom no) (on_board yes)
     (property "Reference" "MCH.SP.5" (id 0) (at 153.67 80.01 0)
       (effects (font (size 1.27 1.27)) (justify left))
@@
   )
   (symbol (lib_name "Spark_gap_19") (lib_id "Mouse_Parts:Spark_gap") (at 135.89 83.82 0) (unit 1)
-    (in_bom yes) (on_board yes)
+    (in_bom no) (on_board yes)
     (property "Reference" "MCH.SP.1" (id 0) (at 130.81 80.01 0)
       (effects (font (size 1.27 1.27)) (justify left))
@@
   )
   (symbol (lib_name "Spark_gap_25") (lib_id "Mouse_Parts:Spark_gap") (at 157.48 134.62 0) (unit 1)
-    (in_bom yes) (on_board yes)
+    (in_bom no) (on_board yes)
     (property "Reference" "MCH.SP.21" (id 0) (at 152.4 128.27 0)
       (effects (font (size 1.27 1.27)) (justify left))
@@
   )
   (symbol (lib_name "Spark_gap_17") (lib_id "Mouse_Parts:Spark_gap") (at 173.99 83.82 0) (unit 1)
-    (in_bom yes) (on_board yes)
+    (in_bom no) (on_board yes)
     (property "Reference" "MCH.SP.8" (id 0) (at 168.91 77.47 0)
       (effects (font (size 1.27 1.27)) (justify left))
@@
   )
   (symbol (lib_name "Spark_gap_22") (lib_id "Mouse_Parts:Spark_gap") (at 165.1 134.62 0) (unit 1)
-    (in_bom yes) (on_board yes)
+    (in_bom no) (on_board yes)
     (property "Reference" "MCH.SP.26" (id 0) (at 160.02 130.81 0)
       (effects (font (size 1.27 1.27)) (justify left))
@@
   )
   (symbol (lib_name "Spark_gap_26") (lib_id "Mouse_Parts:Spark_gap") (at 153.67 134.62 0) (unit 1)
-    (in_bom yes) (on_board yes)
+    (in_bom no) (on_board yes)
     (property "Reference" "MCH.SP.25" (id 0) (at 148.59 130.81 0)
       (effects (font (size 1.27 1.27)) (justify left))
@@
   )
   (symbol (lib_name "Spark_gap_8") (lib_id "Mouse_Parts:Spark_gap") (at 153.67 109.22 0) (unit 1)
-    (in_bom yes) (on_board yes)
+    (in_bom no) (on_board yes)
     (property "Reference" "MCH.SP.13" (id 0) (at 148.59 105.41 0)
       (effects (font (size 1.27 1.27)) (justify left))
@@
   )
   (symbol (lib_name "Spark_gap_7") (lib_id "Mouse_Parts:Spark_gap") (at 181.61 83.82 0) (unit 1)
-    (in_bom yes) (on_board yes)
+    (in_bom no) (on_board yes)
     (property "Reference" "MCH.SP.9" (id 0) (at 176.53 80.01 0)
       (effects (font (size 1.27 1.27)) (justify left))
@@
   )
   (symbol (lib_name "Spark_gap_18") (lib_id "Mouse_Parts:Spark_gap") (at 147.32 83.82 0) (unit 1)
-    (in_bom yes) (on_board yes)
+    (in_bom no) (on_board yes)
     (property "Reference" "MCH.SP.3" (id 0) (at 142.24 80.01 0)
       (effects (font (size 1.27 1.27)) (justify left))
@@
   )
   (symbol (lib_name "Spark_gap_4") (lib_id "Mouse_Parts:Spark_gap") (at 191.77 109.22 0) (unit 1)
-    (in_bom yes) (on_board yes)
+    (in_bom no) (on_board yes)
     (property "Reference" "MCH.SP.20" (id 0) (at 186.69 102.87 0)
       (effects (font (size 1.27 1.27)) (justify left))
@@
   )
   (symbol (lib_name "Spark_gap_11") (lib_id "Mouse_Parts:Spark_gap") (at 168.91 109.22 0) (unit 1)
-    (in_bom yes) (on_board yes)
+    (in_bom no) (on_board yes)
     (property "Reference" "MCH.SP.16" (id 0) (at 163.83 102.87 0)
       (effects (font (size 1.27 1.27)) (justify left))
@@
   )
   (symbol (lib_name "Spark_gap_15") (lib_id "Mouse_Parts:Spark_gap") (at 196.85 83.82 0) (unit 1)
-    (in_bom yes) (on_board yes)
+    (in_bom no) (on_board yes)
     (property "Reference" "MCH.SP.12" (id 0) (at 191.77 77.47 0)
       (effects (font (size 1.27 1.27)) (justify left))
@@
   )
   (symbol (lib_name "Spark_gap_2") (lib_id "Mouse_Parts:Spark_gap") (at 176.53 109.22 0) (unit 1)
-    (in_bom yes) (on_board yes)
+    (in_bom no) (on_board yes)
     (property "Reference" "MCH.SP.17" (id 0) (at 171.45 105.41 0)
       (effects (font (size 1.27 1.27)) (justify left))
@@
   )
   (symbol (lib_id "Mouse_Parts:Fiducial") (at 54.61 53.34 0) (unit 1)
-    (in_bom yes) (on_board yes) (fields_autoplaced)
+    (in_bom no) (on_board yes) (fields_autoplaced)
     (property "Reference" "MCH.FID.1" (id 0) (at 57.15 52.0699 0)
       (effects (font (size 1.27 1.27)) (justify left))
@@
   )
   (symbol (lib_name "Spark_gap_14") (lib_id "Mouse_Parts:Spark_gap") (at 193.04 83.82 0) (unit 1)
-    (in_bom yes) (on_board yes)
+    (in_bom no) (on_board yes)
     (property "Reference" "MCH.SP.11" (id 0) (at 187.96 80.01 0)
       (effects (font (size 1.27 1.27)) (justify left))
@@
   )
   (symbol (lib_id "Mechanical:MountingHole") (at 53.34 69.85 0) (unit 1)
-    (in_bom yes) (on_board yes) (fields_autoplaced)
+    (in_bom no) (on_board yes) (fields_autoplaced)
     (property "Reference" "HOLE.1" (id 0) (at 55.88 68.5799 0)
       (effects (font (size 1.27 1.27)) (justify left))
@@
   )
   (symbol (lib_name "Spark_gap_9") (lib_id "Mouse_Parts:Spark_gap") (at 157.48 109.22 0) (unit 1)
-    (in_bom yes) (on_board yes)
+    (in_bom no) (on_board yes)
     (property "Reference" "MCH.SP.14" (id 0) (at 152.4 102.87 0)
       (effects (font (size 1.27 1.27)) (justify left))
@@
   )
   (symbol (lib_name "Spark_gap_21") (lib_id "Mouse_Parts:Spark_gap") (at 168.91 134.62 0) (unit 1)
-    (in_bom yes) (on_board yes)
+    (in_bom no) (on_board yes)
     (property "Reference" "MCH.SP.22" (id 0) (at 163.83 128.27 0)
       (effects (font (size 1.27 1.27)) (justify left))
@@
   )
   (symbol (lib_id "Mouse_Parts:Coordinate_system_marker") (at 73.66 90.17 0) (unit 1)
-    (in_bom yes) (on_board yes)
+    (in_bom no) (on_board yes)
     (property "Reference" "MCH.LOGO.2" (id 0) (at 67.31 82.55 0)
       (effects (font (size 1.27 1.27)) (justify left))
@@
   )
   (symbol (lib_id "Mouse_Parts:Spark_gap") (at 191.77 134.62 0) (unit 1)
-    (in_bom yes) (on_board yes)
+    (in_bom no) (on_board yes)
     (property "Reference" "MCH.SP.24" (id 0) (at 186.69 128.27 0)
       (effects (font (size 1.27 1.27)) (justify left))
@@
   )
   (symbol (lib_name "Spark_gap_16") (lib_id "Mouse_Parts:Spark_gap") (at 185.42 83.82 0) (unit 1)
-    (in_bom yes) (on_board yes)
+    (in_bom no) (on_board yes)
     (property "Reference" "MCH.SP.10" (id 0) (at 180.34 77.47 0)
       (effects (font (size 1.27 1.27)) (justify left))
@@
   )
   (symbol (lib_name "Spark_gap_12") (lib_id "Mouse_Parts:Spark_gap") (at 162.56 83.82 0) (unit 1)
-    (in_bom yes) (on_board yes)
+    (in_bom no) (on_board yes)
     (property "Reference" "MCH.SP.6" (id 0) (at 157.48 77.47 0)
       (effects (font (size 1.27 1.27)) (justify left))
@@
   )
   (symbol (lib_name "Spark_gap_10") (lib_id "Mouse_Parts:Spark_gap") (at 165.1 109.22 0) (unit 1)
-    (in_bom yes) (on_board yes)
+    (in_bom no) (on_board yes)
     (property "Reference" "MCH.SP.15" (id 0) (at 160.02 105.41 0)
       (effects (font (size 1.27 1.27)) (justify left))
@@
   )
   (symbol (lib_name "Spark_gap_20") (lib_id "Mouse_Parts:Spark_gap") (at 139.7 83.82 0) (unit 1)
-    (in_bom yes) (on_board yes)
+    (in_bom no) (on_board yes)
     (property "Reference" "MCH.SP.2" (id 0) (at 134.62 77.47 0)
       (effects (font (size 1.27 1.27)) (justify left))
@@
   )
   (symbol (lib_name "Spark_gap_23") (lib_id "Mouse_Parts:Spark_gap") (at 180.34 134.62 0) (unit 1)
-    (in_bom yes) (on_board yes)
+    (in_bom no) (on_board yes)
     (property "Reference" "MCH.SP.23" (id 0) (at 175.26 128.27 0)
       (effects (font (size 1.27 1.27)) (justify left))
@@
   )
   (symbol (lib_name "Spark_gap_24") (lib_id "Mouse_Parts:Spark_gap") (at 176.53 134.62 0) (unit 1)
-    (in_bom yes) (on_board yes)
+    (in_bom no) (on_board yes)
     (property "Reference" "MCH.SP.27" (id 0) (at 171.45 130.81 0)
       (effects (font (size 1.27 1.27)) (justify left))
