File: hardware/electronics/QMKMouse/LEDs-SchDoc.kicad_sch (KiCad schematic)
At the start: 20 parts

Commit message: reference 3d model to all components
Parts:
- LED.C.20, LED.C.21, LED.C.23, LED.C.24, LED.C.25, LED.C.26, LED.C.27, LED.C.28: footprint Chip_Passives.PcbLib:0805 -> mouse_part:C_0805
- LED.D.1, LED.D.2, LED.D.3, LED.D.4, LED.D.5, LED.D.6, LED.D.7, LED.D.8: footprint LEDs.PcbLib:IN-PI55TATPRPGPB -> mouse_part:IN-PI55TATPRPGPB
- LED.R.16, LED.R.17, LED.R.18, LED.R.19: footprint Chip_Passives.PcbLib:0805 -> mouse_part:0805
Changed lines of the file:
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@@
       (effects (font (size 1.27 1.27)) (justify left))
     )
-    (property "Footprint" "Chip_Passives.PcbLib:0805" (id 2) (at 199.0852 104.14 0)
+    (property "Footprint" "mouse_part:C_0805" (id 2) (at 199.0852 104.14 0)
       (effects (font (size 1.27 1.27)) hide)
     )
@@
     (property "Reference" "LED.D.7" (id 0) (at 99.06 147.32 0))
     (property "Value" "IN-PI55TATPRPGPB" (id 1) (at 102.87 149.86 0))
-    (property "Footprint" "LEDs.PcbLib:IN-PI55TATPRPGPB" (id 2) (at 88.9 149.86 0)
+    (property "Footprint" "mouse_part:IN-PI55TATPRPGPB" (id 2) (at 88.9 149.86 0)
       (effects (font (size 1.27 1.27)) (justify left top) hide)
     )
@@
       (effects (font (size 1.27 1.27)) (justify left))
     )
-    (property "Footprint" "Chip_Passives.PcbLib:0805" (id 2) (at 199.0852 43.18 0)
+    (property "Footprint" "mouse_part:C_0805" (id 2) (at 199.0852 43.18 0)
       (effects (font (size 1.27 1.27)) hide)
     )
@@
       (effects (font (size 1.27 1.27)) (justify left))
     )
-    (property "Footprint" "Chip_Passives.PcbLib:0805" (id 2) (at 67.0052 104.14 0)
+    (property "Footprint" "mouse_part:C_0805" (id 2) (at 67.0052 104.14 0)
       (effects (font (size 1.27 1.27)) hide)
     )
@@
       (effects (font (size 1.27 1.27)) (justify right))
     )
-    (property "Footprint" "Chip_Passives.PcbLib:0805" (id 2) (at 207.518 151.13 90)
+    (property "Footprint" "mouse_part:0805" (id 2) (at 207.518 151.13 90)
       (effects (font (size 1.27 1.27)) hide)
     )
@@
     (property "Reference" "LED.D.6" (id 0) (at 231.14 116.84 0))
     (property "Value" "IN-PI55TATPRPGPB" (id 1) (at 234.95 119.38 0))
-    (property "Footprint" "LEDs.PcbLib:IN-PI55TATPRPGPB" (id 2) (at 220.98 119.38 0)
+    (property "Footprint" "mouse_part:IN-PI55TATPRPGPB" (id 2) (at 220.98 119.38 0)
       (effects (font (size 1.27 1.27)) (justify left top) hide)
     )
@@
     (property "Reference" "LED.D.2" (id 0) (at 231.14 55.88 0))
     (property "Value" "IN-PI55TATPRPGPB" (id 1) (at 234.95 58.42 0))
-    (property "Footprint" "LEDs.PcbLib:IN-PI55TATPRPGPB" (id 2) (at 220.98 58.42 0)
+    (property "Footprint" "mouse_part:IN-PI55TATPRPGPB" (id 2) (at 220.98 58.42 0)
       (effects (font (size 1.27 1.27)) (justify left top) hide)
     )
@@
       (effects (font (size 1.27 1.27)) (justify left))
     )
-    (property "Footprint" "Chip_Passives.PcbLib:0805" (id 2) (at 199.0852 73.66 0)
+    (property "Footprint" "mouse_part:C_0805" (id 2) (at 199.0852 73.66 0)
       (effects (font (size 1.27 1.27)) hide)
     )
@@
       (effects (font (size 1.27 1.27)) (justify left))
     )
-    (property "Footprint" "Chip_Passives.PcbLib:0805" (id 2) (at 67.0052 43.18 0)
+    (property "Footprint" "mouse_part:C_0805" (id 2) (at 67.0052 43.18 0)
       (effects (font (size 1.27 1.27)) hide)
     )
@@
     (property "Reference" "LED.D.3" (id 0) (at 99.06 86.36 0))
     (property "Value" "IN-PI55TATPRPGPB" (id 1) (at 102.87 88.9 0))
-    (property "Footprint" "LEDs.PcbLib:IN-PI55TATPRPGPB" (id 2) (at 88.9 88.9 0)
+    (property "Footprint" "mouse_part:IN-PI55TATPRPGPB" (id 2) (at 88.9 88.9 0)
       (effects (font (size 1.27 1.27)) (justify left top) hide)
     )
@@
     (property "Reference" "LED.D.5" (id 0) (at 99.06 116.84 0))
     (property "Value" "IN-PI55TATPRPGPB" (id 1) (at 102.87 119.38 0))
-    (property "Footprint" "LEDs.PcbLib:IN-PI55TATPRPGPB" (id 2) (at 88.9 119.38 0)
+    (property "Footprint" "mouse_part:IN-PI55TATPRPGPB" (id 2) (at 88.9 119.38 0)
       (effects (font (size 1.27 1.27)) (justify left top) hide)
     )
@@
       (effects (font (size 1.27 1.27)) (justify left))
     )
-    (property "Footprint" "Chip_Passives.PcbLib:0805" (id 2) (at 199.0852 134.62 0)
+    (property "Footprint" "mouse_part:C_0805" (id 2) (at 199.0852 134.62 0)
       (effects (font (size 1.27 1.27)) hide)
     )
@@
     (property "Reference" "LED.D.4" (id 0) (at 231.14 86.36 0))
     (property "Value" "IN-PI55TATPRPGPB" (id 1) (at 234.95 88.9 0))
-    (property "Footprint" "LEDs.PcbLib:IN-PI55TATPRPGPB" (id 2) (at 220.98 88.9 0)
+    (property "Footprint" "mouse_part:IN-PI55TATPRPGPB" (id 2) (at 220.98 88.9 0)
       (effects (font (size 1.27 1.27)) (justify left top) hide)
     )
@@
     (property "Reference" "LED.R.16" (id 0) (at 93.98 27.94 90))
     (property "Value" "1k 1%" (id 1) (at 93.98 33.02 90))
-    (property "Footprint" "Chip_Passives.PcbLib:0805" (id 2) (at 93.98 28.702 90)
+    (property "Footprint" "mouse_part:0805" (id 2) (at 93.98 28.702 90)
       (effects (font (size 1.27 1.27)) hide)
     )
@@
     (property "Reference" "LED.D.1" (id 0) (at 99.06 55.88 0))
     (property "Value" "IN-PI55TATPRPGPB" (id 1) (at 102.87 58.42 0))
-    (property "Footprint" "LEDs.PcbLib:IN-PI55TATPRPGPB" (id 2) (at 88.9 58.42 0)
+    (property "Footprint" "mouse_part:IN-PI55TATPRPGPB" (id 2) (at 88.9 58.42 0)
       (effects (font (size 1.27 1.27)) (justify left top) hide)
     )
@@
     (property "Reference" "LED.D.8" (id 0) (at 231.14 147.32 0))
     (property "Value" "IN-PI55TATPRPGPB" (id 1) (at 234.95 149.86 0))
-    (property "Footprint" "LEDs.PcbLib:IN-PI55TATPRPGPB" (id 2) (at 220.98 149.86 0)
+    (property "Footprint" "mouse_part:IN-PI55TATPRPGPB" (id 2) (at 220.98 149.86 0)
       (effects (font (size 1.27 1.27)) (justify left top) hide)
     )
@@
       (effects (font (size 1.27 1.27)) (justify right))
     )
-    (property "Footprint" "Chip_Passives.PcbLib:0805" (id 2) (at 75.438 151.13 90)
+    (property "Footprint" "mouse_part:0805" (id 2) (at 75.438 151.13 90)
       (effects (font (size 1.27 1.27)) hide)
     )
@@
       (effects (font (size 1.27 1.27)) (justify left))
     )
-    (property "Footprint" "Chip_Passives.PcbLib:0805" (id 2) (at 67.0052 73.66 0)
+    (property "Footprint" "mouse_part:C_0805" (id 2) (at 67.0052 73.66 0)
       (effects (font (size 1.27 1.27)) hide)
     )
@@
       (effects (font (size 1.27 1.27)) (justify left))
     )
-    (property "Footprint" "Chip_Passives.PcbLib:0805" (id 2) (at 67.0052 134.62 0)
+    (property "Footprint" "mouse_part:C_0805" (id 2) (at 67.0052 134.62 0)
       (effects (font (size 1.27 1.27)) hide)
     )
@@
     (property "Reference" "LED.R.17" (id 0) (at 226.06 27.94 90))
     (property "Value" "1k 1%" (id 1) (at 226.06 33.02 90))
-    (property "Footprint" "Chip_Passives.PcbLib:0805" (id 2) (at 226.06 28.702 90)
-      (effects (font (size 1.27 1.27)) hide)
-    )
+    (property "Footprint" "mouse_part:0805" (id 2) (at 226.06 28.702 90)
+      (effects (font (size 1.27 1.27)) hide)
+    )
