File: hardware/electronics/QMKMouse/ScrollWheel-SchDoc.kicad_sch (KiCad schematic)
At the start: 8 parts

Commit message: reference 3d model to all components
Parts:
- SCW.R.1, SCW.R.2, SCW.R.3, SCW.R.4: footprint Chip_Passives.PcbLib:0805 -> mouse_part:0805
Changed lines of the file:
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@@
       (effects (font (size 1.27 1.27)) (justify right))
     )
-    (property "Footprint" "Chip_Passives.PcbLib:0805" (id 2) (at 80.772 116.84 90)
+    (property "Footprint" "mouse_part:0805" (id 2) (at 80.772 116.84 90)
       (effects (font (size 1.27 1.27)) hide)
     )
@@
       (effects (font (size 1.27 1.27)) (justify right))
     )
-    (property "Footprint" "Chip_Passives.PcbLib:0805" (id 2) (at 80.772 63.5 90)
+    (property "Footprint" "mouse_part:0805" (id 2) (at 80.772 63.5 90)
       (effects (font (size 1.27 1.27)) hide)
     )
@@
       (effects (font (size 1.27 1.27)) (justify right))
     )
-    (property "Footprint" "Chip_Passives.PcbLib:0805" (id 2) (at 131.572 132.08 90)
+    (property "Footprint" "mouse_part:0805" (id 2) (at 131.572 132.08 90)
       (effects (font (size 1.27 1.27)) hide)
     )
@@
       (effects (font (size 1.27 1.27)) (justify right))
     )
-    (property "Footprint" "Chip_Passives.PcbLib:0805" (id 2) (at 131.572 78.74 90)
+    (property "Footprint" "mouse_part:0805" (id 2) (at 131.572 78.74 90)
       (effects (font (size 1.27 1.27)) hide)
     )
